Commit message: Changed R-Axis limits to 360 degrees

File: src/urdf/4dof.urdf (robot description, URDF)
Before this commit: robot 4dof, 6 links, 5 joints
Joints:
- joint r_axis: limit lower=0 upper=3.141592653589793 effort=0 velocity=0.174533 -> lower=0 upper=6.28318530718 effort=0 velocity=0.174533

Commit message: Mounted fixed robot_section_1 at an angle in URDF

File: src/urdf/4dof.urdf (robot description, URDF)
Before this commit: robot 4dof, 6 links, 5 joints
Joints:
- joint base_to_arm_section_1: origin xyz=0 0 0.05 rpy=0 0 0 -> xyz=0 0 0.05 rpy=-0.5 0 0

Commit message: Minor work

File: src/urdf/4dof.urdf (robot description, URDF)
Before this commit: robot 4dof, 6 links, 5 joints
Joints:
- joint base_to_arm_section_1: origin xyz=0 0 0.05 rpy=-0.5 0 0 -> xyz=0 0 0.05 rpy=0 0 0

Commit message: A_section

File: src/urdf/4dof.urdf (robot description, URDF)
Before this commit: robot 4dof, 6 links, 5 joints
Links:
- link arm_section_2: geometry collision mesh filename=meshes/collision/A_section.stl scale=0.003 0.003 0.003; visual mesh filename=meshes/visual/A_section.stl scale=0.003 0.003 0.003
- link arm_section_3: geometry collision mesh filename=meshes/collision/B_section.stl scale=0.003 0.003 0.003; visual mesh filename=meshes/visual/B_section.stl scale=0.003 0.003 0.003
- link arm_section_4: geometry collision mesh filename=meshes/collision/C_axis.stl scale=0.003 0.003 0.003; visual mesh filename=meshes/visual/C_axis.stl scale=0.003 0.003 0.003

Commit message: IK issues

File: src/urdf/4dof.urdf (robot description, URDF)
Before this commit: robot 4dof, 6 links, 5 joints
Links:
- link arm_section_1: geometry collision mesh filename=meshes/collision/R_section_collision.stl scale=0.006 0.006 0.006; visual mesh filename=meshes/visual/R_section.stl scale=0.006 0.006 0.006
- link arm_section_2: geometry collision mesh filename=meshes/collision/A_section_collision.stl scale=0.005 0.005 0.005; visual mesh filename=meshes/visual/A_section.stl scale=0.006 0.006 0.006
- link arm_section_3: geometry collision mesh filename=meshes/collision/B_section_collision.stl scale=0.005 0.005 0.005; visual mesh filename=meshes/visual/B_section.stl scale=0.006 0.006 0.006
- link arm_section_4: geometry collision mesh filename=meshes/collision/C_section_collision.stl scale=0.005 0.005 0.005; visual mesh filename=meshes/visual/C_section.stl scale=0.005 0.005 0.005
- link base: geometry collision mesh filename=meshes/collision/Base_collision.stl scale=0.006 0.006 0.006; visual mesh filename=meshes/visual/Base.stl scale=0.006 0.006 0.006
Joints:
- joint a_axis: axis 1 0 0 -> 0 1 0; limit lower=-1.57079632679 upper=1.57079632679 effort=0 velocity=0.174533 -> lower=-0.77 upper=0.77 effort=0 velocity=0.174533; origin xyz=0 0 0.125 rpy=0 0 0 -> xyz=0 0 0.45 rpy=0 0 0.5
- joint b_axis: axis 1 0 0 -> 0 1 0; limit lower=0 upper=2.8 effort=0 velocity=0.174533 -> lower=-0.6 upper=3.14 effort=0 velocity=0.174533; origin xyz=0 0 0.35 rpy=0 0 0 -> xyz=-0.6 0.2 0.7 rpy=0 0 0
- joint base_to_arm_section_1: origin xyz=0 0 0.05 rpy=0 0 0 -> xyz=0 -0.012 0 rpy=0 0 0
- joint c_axis: axis 1 0 0 -> 0 1 0; limit lower=0 upper=2.8 effort=0 velocity=0.174533 -> lower=-0.6 upper=1.5 effort=0 velocity=0.174533; origin xyz=0 0 0.5 rpy=0 0 0 -> xyz=-0.65 0 -0.55 rpy=0 0 0

Commit message: Updated URDF

File: src/urdf/4dof.urdf (robot description, URDF)
Before this commit: robot onshape, 6 links, 5 joints
Joints:
- joint b_axis: limit lower=-0.6 upper=3.14 effort=0 velocity=0.174533 -> lower=-0.6 upper=2 effort=0 velocity=0.174533; origin xyz=-0.6 0.2 0.7 rpy=0 0 0 -> xyz=-0.65 0.2 0.7 rpy=0 0 0
- joint c_axis: limit lower=-0.6 upper=1.5 effort=0 velocity=0.174533 -> lower=-1.5 upper=1.5 effort=0 velocity=0.174533; origin xyz=-0.65 0 -0.55 rpy=0 0 0 -> xyz=-0.59 0 -0.55 rpy=0 0 0
