Commit message: CAD model into URDF

File: src/urdf/onshape.urdf (robot description, URDF)
Before this commit: robot onshape, 5 links, 4 joints
Links:
- added link arm_section_4, mass 1.0; collision mesh filename=meshes/collision/C_section_collision.stl scale=0.005 0.005 0.005; visual mesh filename=meshes/visual/C_section.stl scale=0.005 0.005 0.005
- link arm_section_2: geometry collision mesh filename=meshes/collision/A_section_collision.stl scale=0.005 0.005 0.005; visual mesh filename=meshes/visual/A_section.stl scale=0.006 0.006 0.006
- link arm_section_3: geometry collision mesh filename=meshes/collision/B_section_collision.stl scale=0.005 0.005 0.005; visual mesh filename=meshes/visual/B_section.stl scale=0.006 0.006 0.006
Joints:
- added joint c_axis: type revolute, parent arm_section_3, child arm_section_4, origin xyz=-0.65 0 -0.55 rpy=0 0 0, axis 0 1 0, limit lower=-0.6 upper=0.6 effort=0 velocity=0.174533
- joint a_axis: axis 0 1 0 -> 0 0.5 0; limit lower=-1.57079632679 upper=1.57079632679 effort=0 velocity=0.174533 -> lower=-0.77 upper=0.77 effort=0 velocity=0.174533; origin xyz=0 0 0.012 rpy=0 0 0 -> xyz=0 0 0.45 rpy=0 0 0.5
- joint b_axis: axis 1 0 0 -> 0 1 0; limit lower=0 upper=2.8 effort=0 velocity=0.174533 -> lower=-0.6 upper=0.6 effort=0 velocity=0.174533; origin xyz=0 0 0 rpy=0 0 0 -> xyz=-0.6 0.2 0.7 rpy=0 0 0

Commit message: Offset for vertical starting pos

File: src/urdf/onshape.urdf (robot description, URDF)
Before this commit: robot onshape, 6 links, 5 joints
Joints:
- joint a_axis: axis 0 0.5 0 -> 0 1 0
- joint b_axis: limit lower=-0.6 upper=0.6 effort=0 velocity=0.174533 -> lower=-0.6 upper=3.14 effort=0 velocity=0.174533
- joint c_axis: limit lower=-0.6 upper=0.6 effort=0 velocity=0.174533 -> lower=-0.6 upper=1.5 effort=0 velocity=0.174533

Commit message: Minor fixes, changing direction of rotation for some axes, and fixing limits in user_controlled for debugging

File: src/urdf/onshape.urdf (robot description, URDF)
Before this commit: robot 4dof, 6 links, 5 joints
Joints:
- joint a_axis: axis 0 1 0 -> 0 -1 0
- joint base_to_arm_section_1: axis 0 0 1 -> 0 0 -1
- joint c_axis: axis 0 1 0 -> 0 -1 0
