Commit message: Final misc.

File: src/urdf/gallbladder.urdf (robot description, URDF)
Before this commit: robot gallbladder, 1 links, 0 joints
Links:
- link gallbladder_link: geometry collision mesh filename=meshes/gallbladder.stl scale=0.005 0.005 0.005; visual mesh filename=meshes/gallbladder.stl scale=0.005 0.005 0.005

Commit message: Final

File: src/urdf/gallbladder.urdf (robot description, URDF)
Before this commit: robot gallbladder, 1 links, 0 joints
Links:
- link gallbladder_link: geometry collision mesh filename=meshes/gallbladder.stl scale=0.0041 0.0041 0.0041; visual mesh filename=meshes/gallbladder.stl scale=0.0041 0.0041 0.0041
