Commit message: Final URDF model + gallbladder +IK updates

File: src/old/urdf/4dof.urdf (robot description, URDF)
Before this commit: robot 4dof, 6 links, 5 joints
Links:
- link arm_section_2: geometry collision cylinder length=0.5 radius=0.05; visual cylinder length=0.35 radius=0.05
- link arm_section_3: geometry collision cylinder length=0.5 radius=0.05; visual cylinder length=0.5 radius=0.05
- link arm_section_4: geometry collision cylinder length=0.25 radius=0.05; visual cylinder length=0.25 radius=0.05
Joints:
- joint a_axis: limit lower=-1.57079632679 upper=1.57079632679 effort=0 velocity=0.174533 -> lower=-1.047 upper=1.39626 effort=0 velocity=0.174533
- joint b_axis: limit lower=0 upper=2.8 effort=0 velocity=0.174533 -> lower=0 upper=2.79253 effort=0 velocity=0.174533
- joint base_to_arm_section_1: origin xyz=0 0 0.05 rpy=0 0 0 -> xyz=0 0 0.05 rpy=-0.5 0 0
- joint c_axis: limit lower=0 upper=2.8 effort=0 velocity=0.174533 -> lower=-1.570796 upper=1.570796 effort=0 velocity=0.174533
- joint r_axis: limit lower=0 upper=6.28318530718 effort=0 velocity=0.174533 -> lower=-3.1415926536 upper=3.1415926536 effort=0 velocity=0.174533

File: src/urdf/4dof.urdf (robot description, URDF)
Before this commit: robot onshape, 6 links, 5 joints
Links:
- link arm_section_1: geometry collision mesh filename=meshes/collision/Bolean ARM1 collision.stl scale=0.006 0.006 0.006; visual mesh filename=meshes/visual/Bolean ARM1.stl scale=0.006 0.006 0.006
- link arm_section_2: geometry collision mesh filename=meshes/collision/Bolean ARM2 collision.stl scale=0.005 0.005 0.005; visual mesh filename=meshes/visual/Bolean ARM2.stl scale=0.006 0.006 0.006
- link base: geometry collision mesh filename=meshes/collision/Bolean Base collision.stl scale=0.006 0.006 0.006; visual mesh filename=meshes/visual/Bolean Base.stl scale=0.006 0.006 0.006
Joints:
- joint a_axis: limit lower=-0.77 upper=0.77 effort=0 velocity=0.174533 -> lower=-1.047 upper=1.39626 effort=0 velocity=0.174533
- joint b_axis: limit lower=-0.6 upper=2 effort=0 velocity=0.174533 -> lower=0 upper=2.79253 effort=0 velocity=0.174533
- joint c_axis: limit lower=-1.5 upper=1.5 effort=0 velocity=0.174533 -> lower=-1.570796 upper=1.570796 effort=0 velocity=0.174533
- joint r_axis: limit lower=0 upper=6.28318530718 effort=0 velocity=0.174533 -> lower=-3.1415926536 upper=3.1415926536 effort=0 velocity=0.174533

File: src/urdf/onshape.urdf (robot description, URDF)
Before this commit: robot 4dof, 5 links, 4 joints
Links:
- added link arm_section_4, mass 1.0; collision mesh filename=meshes/collision/Bolean ARM1 collision.stl scale=0.006 0.006 0.006; visual mesh filename=meshes/visual/Bolean ARM1.stl scale=0.006 0.006 0.006
- link arm_section_2: geometry collision mesh filename=meshes/collision/Bolean ARM3 collision.stl scale=0.006 0.006 0.006; visual mesh filename=meshes/visual/Bolean ARM3.stl scale=0.006 0.006 0.006
- link arm_section_3: geometry collision mesh filename=meshes/collision/Bolean ARM2 collision.stl scale=0.006 0.006 0.006; visual mesh filename=meshes/visual/Bolean ARM2.stl scale=0.006 0.006 0.006
Joints:
- added joint a_axis: type revolute, parent arm_section_3, child arm_section_4, origin xyz=0 0.215 0.88 rpy=0 0 0, axis 0 1 0, limit lower=-1.570796 upper=1.570796 effort=0 velocity=0.174533
- joint b_axis: axis 0 1 0 -> 0 -1 0; origin xyz=0 0 0.8 rpy=0 0 0 -> xyz=-0.17 0 0.96 rpy=0 0 0
- joint base_to_arm_section_1: axis (none) -> 0 0 1; limit (none) -> lower=-1.047 upper=1.047 effort=0 velocity=0.174533; origin xyz=0 0 0.05 rpy=0 0 0 -> xyz=0 0 0.15 rpy=0 0 0; type fixed -> revolute
- joint r_axis: axis 0 0 1 -> (none); limit lower=-3.1415926536 upper=3.1415926536 effort=0 velocity=0.174533 -> (none); origin xyz=0 0 0 rpy=0 0 0 -> xyz=0 0 0.03 rpy=0 0 0; type revolute -> fixed
